Commit message: Refactor URDF model: Update link dimensions, masses, and joint configurations for improved accuracy and performance

File: test.urdf (robot description, URDF)
Before this commit: robot pepe, 5 links, 4 joints
Links:
- removed link 12
- removed link 13
- added link 115, mass 0.019648212092834492; collision cylinder length=1.4548268328664802 radius=0.0655663384369527; visual cylinder length=1.4548268328664802 radius=0.0655663384369527
- added link 18, mass 0.019648212092834492; collision cylinder length=1.4548268328664802 radius=0.0655663384369527; visual cylinder length=1.4548268328664802 radius=0.0655663384369527
- added link 210, mass 0.34614496777664583; collision cylinder length=1.538953104581494 radius=0.2675724416847266; visual cylinder length=1.538953104581494 radius=0.2675724416847266
- added link 211, mass 0.34614496777664583; collision cylinder length=1.538953104581494 radius=0.2675724416847266; visual cylinder length=1.538953104581494 radius=0.2675724416847266
- added link 216, mass 0.34614496777664583; collision cylinder length=1.538953104581494 radius=0.2675724416847266; visual cylinder length=1.538953104581494 radius=0.2675724416847266
- added link 217, mass 0.34614496777664583; collision cylinder length=1.538953104581494 radius=0.2675724416847266; visual cylinder length=1.538953104581494 radius=0.2675724416847266
- added link 218, mass 0.34614496777664583; collision cylinder length=1.538953104581494 radius=0.2675724416847266; visual cylinder length=1.538953104581494 radius=0.2675724416847266
- added link 22, mass 0.34614496777664583; collision cylinder length=1.538953104581494 radius=0.2675724416847266; visual cylinder length=1.538953104581494 radius=0.2675724416847266
- added link 23, mass 0.34614496777664583; collision cylinder length=1.538953104581494 radius=0.2675724416847266; visual cylinder length=1.538953104581494 radius=0.2675724416847266
- added link 29, mass 0.34614496777664583; collision cylinder length=1.538953104581494 radius=0.2675724416847266; visual cylinder length=1.538953104581494 radius=0.2675724416847266
- added link 312, mass 1.2766658170365746; collision cylinder length=1.6430092711441677 radius=0.4973288710518091; visual cylinder length=1.6430092711441677 radius=0.4973288710518091
- added link 313, mass 1.2766658170365746; collision cylinder length=1.6430092711441677 radius=0.4973288710518091; visual cylinder length=1.6430092711441677 radius=0.4973288710518091
- added link 314, mass 1.2766658170365746; collision cylinder length=1.6430092711441677 radius=0.4973288710518091; visual cylinder length=1.6430092711441677 radius=0.4973288710518091
- added link 319, mass 1.2766658170365746; collision cylinder length=1.6430092711441677 radius=0.4973288710518091; visual cylinder length=1.6430092711441677 radius=0.4973288710518091
- added link 320, mass 1.2766658170365746; collision cylinder length=1.6430092711441677 radius=0.4973288710518091; visual cylinder length=1.6430092711441677 radius=0.4973288710518091
- added link 321, mass 1.2766658170365746; collision cylinder length=1.6430092711441677 radius=0.4973288710518091; visual cylinder length=1.6430092711441677 radius=0.4973288710518091
- added link 35, mass 1.2766658170365746; collision cylinder length=1.6430092711441677 radius=0.4973288710518091; visual cylinder length=1.6430092711441677 radius=0.4973288710518091
- added link 36, mass 1.2766658170365746; collision cylinder length=1.6430092711441677 radius=0.4973288710518091; visual cylinder length=1.6430092711441677 radius=0.4973288710518091
- added link 37, mass 1.2766658170365746; collision cylinder length=1.6430092711441677 radius=0.4973288710518091; visual cylinder length=1.6430092711441677 radius=0.4973288710518091
- added link 422, mass 0.033920912927282665; collision cylinder length=0.03891865824642626 radius=0.5267201102531426; visual cylinder length=0.03891865824642626 radius=0.5267201102531426
- added link 423, mass 0.033920912927282665; collision cylinder length=0.03891865824642626 radius=0.5267201102531426; visual cylinder length=0.03891865824642626 radius=0.5267201102531426
- added link 424, mass 0.033920912927282665; collision cylinder length=0.03891865824642626 radius=0.5267201102531426; visual cylinder length=0.03891865824642626 radius=0.5267201102531426
- link 0: mass 0.08882193011447076 -> 0.0025394449091724614; geometry collision cylinder length=0.6670524266296746 radius=0.03481083792940143; visual cylinder length=0.6670524266296746 radius=0.03481083792940143
- link 11: mass 1.3629571017358157 -> 0.019648212092834492; geometry collision cylinder length=1.4548268328664802 radius=0.0655663384369527; visual cylinder length=1.4548268328664802 radius=0.0655663384369527
- link 24: mass 0.00927975494390793 -> 0.34614496777664583; geometry collision cylinder length=1.538953104581494 radius=0.2675724416847266; visual cylinder length=1.538953104581494 radius=0.2675724416847266
Joints:
- removed joint 12_to_0
- removed joint 13_to_0
- removed joint 24_to_0
- added joint 115_to_0: type revolute, parent 0, child 115, origin xyz=0.6930658259739374 0.6883278041819902 0.0 rpy=22.025669307485494 0.6334335364638696 4.596309397093748, axis 1 0 0, limit lower=3.1415 upper=-3.1415 effort=1 velocity=1
- added joint 18_to_0: type revolute, parent 0, child 18, origin xyz=0.6930658259739374 0.6883278041819902 0.0 rpy=16.519251980614122 0.6334335364638696 4.596309397093748, axis 1 0 0, limit lower=3.1415 upper=-3.1415 effort=1 velocity=1
- added joint 210_to_18: type revolute, parent 18, child 210, origin xyz=0.3136201001316125 0.8683193192565382 0.36803804984502797 rpy=10.289241821405692 2.1728993128546867 5.329896742733081, axis 1 0 0, limit lower=3.1415 upper=-3.1415 effort=1 velocity=1
- added joint 211_to_18: type revolute, parent 18, child 211, origin xyz=0.3136201001316125 0.8683193192565382 0.36803804984502797 rpy=13.71898909520759 2.1728993128546867 5.329896742733081, axis 1 0 0, limit lower=3.1415 upper=-3.1415 effort=1 velocity=1
- added joint 216_to_115: type revolute, parent 115, child 216, origin xyz=0.3136201001316125 0.8683193192565382 0.36803804984502797 rpy=6.859494547603795 2.1728993128546867 5.329896742733081, axis 1 0 0, limit lower=3.1415 upper=-3.1415 effort=1 velocity=1
- added joint 217_to_115: type revolute, parent 115, child 217, origin xyz=0.3136201001316125 0.8683193192565382 0.36803804984502797 rpy=10.289241821405692 2.1728993128546867 5.329896742733081, axis 1 0 0, limit lower=3.1415 upper=-3.1415 effort=1 velocity=1
- added joint 218_to_115: type revolute, parent 115, child 218, origin xyz=0.3136201001316125 0.8683193192565382 0.36803804984502797 rpy=13.71898909520759 2.1728993128546867 5.329896742733081, axis 1 0 0, limit lower=3.1415 upper=-3.1415 effort=1 velocity=1
- added joint 22_to_11: type revolute, parent 11, child 22, origin xyz=0.3136201001316125 0.8683193192565382 0.36803804984502797 rpy=6.859494547603795 2.1728993128546867 5.329896742733081, axis 1 0 0, limit lower=3.1415 upper=-3.1415 effort=1 velocity=1
- added joint 23_to_11: type revolute, parent 11, child 23, origin xyz=0.3136201001316125 0.8683193192565382 0.36803804984502797 rpy=10.289241821405692 2.1728993128546867 5.329896742733081, axis 1 0 0, limit lower=3.1415 upper=-3.1415 effort=1 velocity=1
- added joint 24_to_11: type revolute, parent 11, child 24, origin xyz=0.3136201001316125 0.8683193192565382 0.36803804984502797 rpy=13.71898909520759 2.1728993128546867 5.329896742733081, axis 1 0 0, limit lower=3.1415 upper=-3.1415 effort=1 velocity=1
- added joint 29_to_18: type revolute, parent 18, child 29, origin xyz=0.3136201001316125 0.8683193192565382 0.36803804984502797 rpy=6.859494547603795 2.1728993128546867 5.329896742733081, axis 1 0 0, limit lower=3.1415 upper=-3.1415 effort=1 velocity=1
- added joint 312_to_18: type revolute, parent 18, child 312, origin xyz=0.0 0.7518053736316033 0.6285818416300548 rpy=2.3492450703415018 4.30016643414523 1.869375619771222, axis 1 0 0, limit lower=3.1415 upper=-3.1415 effort=1 velocity=1
- added joint 313_to_18: type revolute, parent 18, child 313, origin xyz=0.0 0.7518053736316033 0.6285818416300548 rpy=2.819094084409802 4.30016643414523 1.869375619771222, axis 1 0 0, limit lower=3.1415 upper=-3.1415 effort=1 velocity=1
- added joint 314_to_18: type revolute, parent 18, child 314, origin xyz=0.0 0.7518053736316033 0.6285818416300548 rpy=3.2889430984781023 4.30016643414523 1.869375619771222, axis 1 0 0, limit lower=3.1415 upper=-3.1415 effort=1 velocity=1
- added joint 319_to_115: type revolute, parent 115, child 319, origin xyz=0.0 0.7518053736316033 0.6285818416300548 rpy=2.3492450703415018 4.30016643414523 1.869375619771222, axis 1 0 0, limit lower=3.1415 upper=-3.1415 effort=1 velocity=1
- added joint 320_to_115: type revolute, parent 115, child 320, origin xyz=0.0 0.7518053736316033 0.6285818416300548 rpy=2.819094084409802 4.30016643414523 1.869375619771222, axis 1 0 0, limit lower=3.1415 upper=-3.1415 effort=1 velocity=1
- added joint 321_to_115: type revolute, parent 115, child 321, origin xyz=0.0 0.7518053736316033 0.6285818416300548 rpy=3.2889430984781023 4.30016643414523 1.869375619771222, axis 1 0 0, limit lower=3.1415 upper=-3.1415 effort=1 velocity=1
- added joint 35_to_11: type revolute, parent 11, child 35, origin xyz=0.0 0.7518053736316033 0.6285818416300548 rpy=2.3492450703415018 4.30016643414523 1.869375619771222, axis 1 0 0, limit lower=3.1415 upper=-3.1415 effort=1 velocity=1
- added joint 36_to_11: type revolute, parent 11, child 36, origin xyz=0.0 0.7518053736316033 0.6285818416300548 rpy=2.819094084409802 4.30016643414523 1.869375619771222, axis 1 0 0, limit lower=3.1415 upper=-3.1415 effort=1 velocity=1
- added joint 37_to_11: type revolute, parent 11, child 37, origin xyz=0.0 0.7518053736316033 0.6285818416300548 rpy=3.2889430984781023 4.30016643414523 1.869375619771222, axis 1 0 0, limit lower=3.1415 upper=-3.1415 effort=1 velocity=1
- added joint 422_to_0: type revolute, parent 0, child 422, origin xyz=0.5108092731201483 0.4602385347308995 0.5410186617412392 rpy=27.201617517057805 3.4598168681769876 1.0178181328046516, axis 1 0 0, limit lower=3.1415 upper=-3.1415 effort=1 velocity=1
- added joint 423_to_0: type revolute, parent 0, child 423, origin xyz=0.5108092731201483 0.4602385347308995 0.5410186617412392 rpy=32.64194102046936 3.4598168681769876 1.0178181328046516, axis 1 0 0, limit lower=3.1415 upper=-3.1415 effort=1 velocity=1
- added joint 424_to_0: type revolute, parent 0, child 424, origin xyz=0.5108092731201483 0.4602385347308995 0.5410186617412392 rpy=38.08226452388092 3.4598168681769876 1.0178181328046516, axis 1 0 0, limit lower=3.1415 upper=-3.1415 effort=1 velocity=1
- joint 11_to_0: axis 0 0 1 -> 1 0 0; origin xyz=0.13758607675745194 0.9350807390271525 0.7734982986138889 rpy=1.1448832225386056 4.335027266637536 1.6623373384868418 -> xyz=0.6930658259739374 0.6883278041819902 0.0 rpy=11.012834653742747 0.6334335364638696 4.596309397093748
