Commit message: Refactor URDF model: Replace cylinder geometries with box geometries, update masses and inertial properties, and rename links and joints for clarity and consistency.

File: temp0.urdf (robot description, URDF)
Before this commit: robot pepe, 11 links, 10 joints
Links:
- removed link 12
- removed link 23
- removed link 34
- removed link 35
- removed link 36
- removed link 410
- removed link 57
- removed link 58
- removed link 59
- added link 210, mass 1.469920476335954; collision box size=1.4246017300798173 1.4246017300798173 0.9221828122795191; visual box size=1.4246017300798173 1.4246017300798173 0.9221828122795191
- added link 22, mass 1.469920476335954; collision box size=1.4246017300798173 1.4246017300798173 0.9221828122795191; visual box size=1.4246017300798173 1.4246017300798173 0.9221828122795191
- added link 26, mass 1.469920476335954; collision box size=1.4246017300798173 1.4246017300798173 0.9221828122795191; visual box size=1.4246017300798173 1.4246017300798173 0.9221828122795191
- added link 314, mass 0.0031971122794980603; collision box size=0.05386615729813338 0.05386615729813338 1.40293004860074; visual box size=0.05386615729813338 0.05386615729813338 1.40293004860074
- added link 411, mass 0.5738342783156067; collision box size=0.7565417280677009 0.7565417280677009 1.2765294304110082; visual box size=0.7565417280677009 0.7565417280677009 1.2765294304110082
- added link 412, mass 0.5738342783156067; collision box size=0.7565417280677009 0.7565417280677009 1.2765294304110082; visual box size=0.7565417280677009 0.7565417280677009 1.2765294304110082
- added link 413, mass 0.5738342783156067; collision box size=0.7565417280677009 0.7565417280677009 1.2765294304110082; visual box size=0.7565417280677009 0.7565417280677009 1.2765294304110082
- added link 43, mass 0.5738342783156067; collision box size=0.7565417280677009 0.7565417280677009 1.2765294304110082; visual box size=0.7565417280677009 0.7565417280677009 1.2765294304110082
- added link 44, mass 0.5738342783156067; collision box size=0.7565417280677009 0.7565417280677009 1.2765294304110082; visual box size=0.7565417280677009 0.7565417280677009 1.2765294304110082
- added link 45, mass 0.5738342783156067; collision box size=0.7565417280677009 0.7565417280677009 1.2765294304110082; visual box size=0.7565417280677009 0.7565417280677009 1.2765294304110082
- added link 47, mass 0.5738342783156067; collision box size=0.7565417280677009 0.7565417280677009 1.2765294304110082; visual box size=0.7565417280677009 0.7565417280677009 1.2765294304110082
- added link 48, mass 0.5738342783156067; collision box size=0.7565417280677009 0.7565417280677009 1.2765294304110082; visual box size=0.7565417280677009 0.7565417280677009 1.2765294304110082
- added link 49, mass 0.5738342783156067; collision box size=0.7565417280677009 0.7565417280677009 1.2765294304110082; visual box size=0.7565417280677009 0.7565417280677009 1.2765294304110082
- link 0: mass 0.40980165276897973 -> 0.016562221436832083; geometry collision cylinder length=0.009057844543907345 radius=0.7629075725563641; visual cylinder length=0.009057844543907345 radius=0.7629075725563641
- link 11: mass 0.1498647321309275 -> 0.05843720197760504; geometry collision box size=0.2525164925054415 0.2525164925054415 1.1668634471253905; visual box size=0.2525164925054415 0.2525164925054415 1.1668634471253905
Joints:
- removed joint 12_to_0
- removed joint 23_to_0
- removed joint 34_to_23
- removed joint 35_to_23
- removed joint 36_to_23
- removed joint 410_to_0
- removed joint 57_to_23
- removed joint 58_to_23
- removed joint 59_to_23
- added joint 210_to_11: type revolute, parent 11, child 210, origin xyz=0.9999 0.44850076168047337 0.26165231731438815 rpy=5.487441334901619 2.2733772407708366 1.2236154125144392, axis 1 0 0, limit lower=3.1415 upper=-3.1415 effort=1 velocity=1
- added joint 22_to_11: type revolute, parent 11, child 22, origin xyz=0.9999 0.44850076168047337 0.26165231731438815 rpy=2.7437206674508094 2.2733772407708366 1.2236154125144392, axis 1 0 0, limit lower=3.1415 upper=-3.1415 effort=1 velocity=1
- added joint 26_to_11: type revolute, parent 11, child 26, origin xyz=0.9999 0.44850076168047337 0.26165231731438815 rpy=4.115581001176214 2.2733772407708366 1.2236154125144392, axis 1 0 0, limit lower=3.1415 upper=-3.1415 effort=1 velocity=1
- added joint 314_to_0: type revolute, parent 0, child 314, origin xyz=0.533500759190922 0.9505003347875978 0.46205782805718615 rpy=6.62830480933661 1.0083435977602198 3.580774287573142, axis 0 1 0, limit lower=3.1415 upper=-3.1415 effort=1 velocity=1
- added joint 411_to_210: type revolute, parent 210, child 411, origin xyz=0.5320185349151316 0.5318004392589183 0.9158069914079802 rpy=9.854211496034896 3.5932832422801697 0.546684880848328, axis 0 1 0, limit lower=3.1415 upper=-3.1415 effort=1 velocity=1
- added joint 412_to_210: type revolute, parent 210, child 412, origin xyz=0.5320185349151316 0.5318004392589183 0.9158069914079802 rpy=14.781317244052344 3.5932832422801697 0.546684880848328, axis 0 1 0, limit lower=3.1415 upper=-3.1415 effort=1 velocity=1
- added joint 413_to_210: type revolute, parent 210, child 413, origin xyz=0.5320185349151316 0.5318004392589183 0.9158069914079802 rpy=19.708422992069792 3.5932832422801697 0.546684880848328, axis 0 1 0, limit lower=3.1415 upper=-3.1415 effort=1 velocity=1
- added joint 43_to_22: type revolute, parent 22, child 43, origin xyz=0.5320185349151316 0.5318004392589183 0.9158069914079802 rpy=9.854211496034896 3.5932832422801697 0.546684880848328, axis 0 1 0, limit lower=3.1415 upper=-3.1415 effort=1 velocity=1
- added joint 44_to_22: type revolute, parent 22, child 44, origin xyz=0.5320185349151316 0.5318004392589183 0.9158069914079802 rpy=14.781317244052344 3.5932832422801697 0.546684880848328, axis 0 1 0, limit lower=3.1415 upper=-3.1415 effort=1 velocity=1
- added joint 45_to_22: type revolute, parent 22, child 45, origin xyz=0.5320185349151316 0.5318004392589183 0.9158069914079802 rpy=19.708422992069792 3.5932832422801697 0.546684880848328, axis 0 1 0, limit lower=3.1415 upper=-3.1415 effort=1 velocity=1
- added joint 47_to_26: type revolute, parent 26, child 47, origin xyz=0.5320185349151316 0.5318004392589183 0.9158069914079802 rpy=9.854211496034896 3.5932832422801697 0.546684880848328, axis 0 1 0, limit lower=3.1415 upper=-3.1415 effort=1 velocity=1
- added joint 48_to_26: type revolute, parent 26, child 48, origin xyz=0.5320185349151316 0.5318004392589183 0.9158069914079802 rpy=14.781317244052344 3.5932832422801697 0.546684880848328, axis 0 1 0, limit lower=3.1415 upper=-3.1415 effort=1 velocity=1
- added joint 49_to_26: type revolute, parent 26, child 49, origin xyz=0.5320185349151316 0.5318004392589183 0.9158069914079802 rpy=19.708422992069792 3.5932832422801697 0.546684880848328, axis 0 1 0, limit lower=3.1415 upper=-3.1415 effort=1 velocity=1
- joint 11_to_0: origin xyz=0.20567582006374824 0.31968346875035925 0.8493649811485663 rpy=6.194556496946603 0.21335447278590858 4.444530471048643 -> xyz=0.9739137415158122 0.9999 0.9753723564264214 rpy=6.623305055309696 2.0355958124422133 1.1957713899188829

File: test.urdf (robot description, URDF)
Before this commit: robot pepe, 25 links, 24 joints
Links:
- removed link 115
- removed link 18
- removed link 211
- removed link 216
- removed link 217
- removed link 218
- removed link 23
- removed link 24
- removed link 29
- removed link 312
- removed link 313
- removed link 319
- removed link 320
- removed link 321
- removed link 35
- removed link 36
- removed link 37
- removed link 422
- removed link 423
- removed link 424
- added link 26, mass 1.469920476335954; collision box size=1.4246017300798173 1.4246017300798173 0.9221828122795191; visual box size=1.4246017300798173 1.4246017300798173 0.9221828122795191
- added link 411, mass 0.5738342783156067; collision box size=0.7565417280677009 0.7565417280677009 1.2765294304110082; visual box size=0.7565417280677009 0.7565417280677009 1.2765294304110082
- added link 412, mass 0.5738342783156067; collision box size=0.7565417280677009 0.7565417280677009 1.2765294304110082; visual box size=0.7565417280677009 0.7565417280677009 1.2765294304110082
- added link 413, mass 0.5738342783156067; collision box size=0.7565417280677009 0.7565417280677009 1.2765294304110082; visual box size=0.7565417280677009 0.7565417280677009 1.2765294304110082
- added link 43, mass 0.5738342783156067; collision box size=0.7565417280677009 0.7565417280677009 1.2765294304110082; visual box size=0.7565417280677009 0.7565417280677009 1.2765294304110082
- added link 44, mass 0.5738342783156067; collision box size=0.7565417280677009 0.7565417280677009 1.2765294304110082; visual box size=0.7565417280677009 0.7565417280677009 1.2765294304110082
- added link 45, mass 0.5738342783156067; collision box size=0.7565417280677009 0.7565417280677009 1.2765294304110082; visual box size=0.7565417280677009 0.7565417280677009 1.2765294304110082
- added link 47, mass 0.5738342783156067; collision box size=0.7565417280677009 0.7565417280677009 1.2765294304110082; visual box size=0.7565417280677009 0.7565417280677009 1.2765294304110082
- added link 48, mass 0.5738342783156067; collision box size=0.7565417280677009 0.7565417280677009 1.2765294304110082; visual box size=0.7565417280677009 0.7565417280677009 1.2765294304110082
- added link 49, mass 0.5738342783156067; collision box size=0.7565417280677009 0.7565417280677009 1.2765294304110082; visual box size=0.7565417280677009 0.7565417280677009 1.2765294304110082
- link 0: mass 0.0025394449091724614 -> 0.016562221436832083; geometry collision box size=1.5258151451127282 1.5258151451127282 0.009057844543907345; visual box size=1.5258151451127282 1.5258151451127282 0.009057844543907345
- link 11: mass 0.019648212092834492 -> 0.05843720197760504; geometry collision box size=0.2525164925054415 0.2525164925054415 1.1668634471253905; visual box size=0.2525164925054415 0.2525164925054415 1.1668634471253905
- link 210: mass 0.34614496777664583 -> 1.469920476335954; geometry collision box size=1.4246017300798173 1.4246017300798173 0.9221828122795191; visual box size=1.4246017300798173 1.4246017300798173 0.9221828122795191
- link 22: mass 0.34614496777664583 -> 1.469920476335954; geometry collision box size=1.4246017300798173 1.4246017300798173 0.9221828122795191; visual box size=1.4246017300798173 1.4246017300798173 0.9221828122795191
- link 314: mass 1.2766658170365746 -> 0.0031971122794980603; geometry collision box size=0.05386615729813338 0.05386615729813338 1.40293004860074; visual box size=0.05386615729813338 0.05386615729813338 1.40293004860074
Joints:
- removed joint 115_to_0
- removed joint 18_to_0
- removed joint 210_to_18
- removed joint 211_to_18
- removed joint 216_to_115
- removed joint 217_to_115
- removed joint 218_to_115
- removed joint 23_to_11
- removed joint 24_to_11
- removed joint 29_to_18
- removed joint 312_to_18
- removed joint 313_to_18
- removed joint 314_to_18
- removed joint 319_to_115
- removed joint 320_to_115
- removed joint 321_to_115
- removed joint 35_to_11
- removed joint 36_to_11
- removed joint 37_to_11
- removed joint 422_to_0
- removed joint 423_to_0
- removed joint 424_to_0
- added joint 210_to_11: type revolute, parent 11, child 210, origin xyz=0.9999 0.44850076168047337 0.26165231731438815 rpy=5.487441334901619 2.2733772407708366 1.2236154125144392, axis 1 0 0, limit lower=3.1415 upper=-3.1415 effort=1 velocity=1
- added joint 26_to_11: type revolute, parent 11, child 26, origin xyz=0.9999 0.44850076168047337 0.26165231731438815 rpy=4.115581001176214 2.2733772407708366 1.2236154125144392, axis 1 0 0, limit lower=3.1415 upper=-3.1415 effort=1 velocity=1
- added joint 314_to_0: type revolute, parent 0, child 314, origin xyz=0.533500759190922 0.9505003347875978 0.46205782805718615 rpy=6.62830480933661 1.0083435977602198 3.580774287573142, axis 0 1 0, limit lower=3.1415 upper=-3.1415 effort=1 velocity=1
- added joint 411_to_210: type revolute, parent 210, child 411, origin xyz=0.5320185349151316 0.5318004392589183 0.9158069914079802 rpy=9.854211496034896 3.5932832422801697 0.546684880848328, axis 0 1 0, limit lower=3.1415 upper=-3.1415 effort=1 velocity=1
- added joint 412_to_210: type revolute, parent 210, child 412, origin xyz=0.5320185349151316 0.5318004392589183 0.9158069914079802 rpy=14.781317244052344 3.5932832422801697 0.546684880848328, axis 0 1 0, limit lower=3.1415 upper=-3.1415 effort=1 velocity=1
- added joint 413_to_210: type revolute, parent 210, child 413, origin xyz=0.5320185349151316 0.5318004392589183 0.9158069914079802 rpy=19.708422992069792 3.5932832422801697 0.546684880848328, axis 0 1 0, limit lower=3.1415 upper=-3.1415 effort=1 velocity=1
- added joint 43_to_22: type revolute, parent 22, child 43, origin xyz=0.5320185349151316 0.5318004392589183 0.9158069914079802 rpy=9.854211496034896 3.5932832422801697 0.546684880848328, axis 0 1 0, limit lower=3.1415 upper=-3.1415 effort=1 velocity=1
- added joint 44_to_22: type revolute, parent 22, child 44, origin xyz=0.5320185349151316 0.5318004392589183 0.9158069914079802 rpy=14.781317244052344 3.5932832422801697 0.546684880848328, axis 0 1 0, limit lower=3.1415 upper=-3.1415 effort=1 velocity=1
- added joint 45_to_22: type revolute, parent 22, child 45, origin xyz=0.5320185349151316 0.5318004392589183 0.9158069914079802 rpy=19.708422992069792 3.5932832422801697 0.546684880848328, axis 0 1 0, limit lower=3.1415 upper=-3.1415 effort=1 velocity=1
- added joint 47_to_26: type revolute, parent 26, child 47, origin xyz=0.5320185349151316 0.5318004392589183 0.9158069914079802 rpy=9.854211496034896 3.5932832422801697 0.546684880848328, axis 0 1 0, limit lower=3.1415 upper=-3.1415 effort=1 velocity=1
- added joint 48_to_26: type revolute, parent 26, child 48, origin xyz=0.5320185349151316 0.5318004392589183 0.9158069914079802 rpy=14.781317244052344 3.5932832422801697 0.546684880848328, axis 0 1 0, limit lower=3.1415 upper=-3.1415 effort=1 velocity=1
- added joint 49_to_26: type revolute, parent 26, child 49, origin xyz=0.5320185349151316 0.5318004392589183 0.9158069914079802 rpy=19.708422992069792 3.5932832422801697 0.546684880848328, axis 0 1 0, limit lower=3.1415 upper=-3.1415 effort=1 velocity=1
- joint 11_to_0: axis 1 0 0 -> 0 0 1; origin xyz=0.6930658259739374 0.6883278041819902 0.0 rpy=11.012834653742747 0.6334335364638696 4.596309397093748 -> xyz=0.9739137415158122 0.9999 0.9753723564264214 rpy=6.623305055309696 2.0355958124422133 1.1957713899188829
- joint 22_to_11: origin xyz=0.3136201001316125 0.8683193192565382 0.36803804984502797 rpy=6.859494547603795 2.1728993128546867 5.329896742733081 -> xyz=0.9999 0.44850076168047337 0.26165231731438815 rpy=2.7437206674508094 2.2733772407708366 1.2236154125144392

Commit message: Enhance simulation with directional sensing and update URDF models
- Added a method to calculate the direction signal for creatures in the simulation, allowing them to sense their orientation towards a peak.
- Modified the `update_motors` method to incorporate sensor signals into motor control for improved responsiveness.
- Updated the URDF files (`temp0.urdf` and `test.urdf`) to replace box geometries with cylinders, adjusting dimensions and masses accordingly for better physical representation.
- Removed redundant links and joints in the URDF files to streamline the robot model.

File: temp0.urdf (robot description, URDF)
Before this commit: robot pepe, 15 links, 14 joints
Links:
- removed link 210
- removed link 26
- removed link 314
- removed link 411
- removed link 412
- removed link 413
- removed link 43
- removed link 44
- removed link 45
- removed link 47
- removed link 48
- removed link 49
- added link 23, mass 0.3931597829033822; collision cylinder length=0.42493009252937664 radius=0.5426888053709441; visual cylinder length=0.42493009252937664 radius=0.5426888053709441
- added link 24, mass 0.3931597829033822; collision cylinder length=0.42493009252937664 radius=0.5426888053709441; visual cylinder length=0.42493009252937664 radius=0.5426888053709441
- link 0: mass 0.016562221436832083 -> 0.003919360339250734; geometry collision cylinder length=1.442823644237529 radius=0.02940532847591959; visual cylinder length=1.442823644237529 radius=0.02940532847591959
- link 11: mass 0.05843720197760504 -> 0.007085101111084106; geometry collision cylinder length=0.039176576910777916 radius=0.23993016166726788; visual cylinder length=0.039176576910777916 radius=0.23993016166726788
- link 22: mass 1.469920476335954 -> 0.3931597829033822; geometry collision cylinder length=0.42493009252937664 radius=0.5426888053709441; visual cylinder length=0.42493009252937664 radius=0.5426888053709441
Joints:
- removed joint 210_to_11
- removed joint 26_to_11
- removed joint 314_to_0
- removed joint 411_to_210
- removed joint 412_to_210
- removed joint 413_to_210
- removed joint 43_to_22
- removed joint 44_to_22
- removed joint 45_to_22
- removed joint 47_to_26
- removed joint 48_to_26
- removed joint 49_to_26
- added joint 23_to_11: type revolute, parent 11, child 23, origin xyz=0.18865344949164164 0.9109936564573404 0.3734537855485758 rpy=18.15343757858938 5.186843867187901 0.0, axis 0 0 1, limit lower=3.1415 upper=-3.1415 effort=1 velocity=1
- added joint 24_to_11: type revolute, parent 11, child 24, origin xyz=0.18865344949164164 0.9109936564573404 0.3734537855485758 rpy=24.204583438119172 5.186843867187901 0.0, axis 0 0 1, limit lower=3.1415 upper=-3.1415 effort=1 velocity=1
- joint 11_to_0: origin xyz=0.9739137415158122 0.9999 0.9753723564264214 rpy=6.623305055309696 2.0355958124422133 1.1957713899188829 -> xyz=0.8100042387937797 0.8497545831898448 0.8428329151479883 rpy=4.726851421616899 2.1332596079635504 5.241707572172651
- joint 22_to_11: axis 1 0 0 -> 0 0 1; origin xyz=0.9999 0.44850076168047337 0.26165231731438815 rpy=2.7437206674508094 2.2733772407708366 1.2236154125144392 -> xyz=0.18865344949164164 0.9109936564573404 0.3734537855485758 rpy=12.102291719059586 5.186843867187901 0.0

File: test.urdf (robot description, URDF)
Before this commit: robot pepe, 15 links, 14 joints
Links:
- removed link 210
- removed link 26
- removed link 314
- removed link 411
- removed link 412
- removed link 413
- removed link 43
- removed link 44
- removed link 45
- removed link 47
- removed link 48
- removed link 49
- added link 23, mass 0.3931597829033822; collision cylinder length=0.42493009252937664 radius=0.5426888053709441; visual cylinder length=0.42493009252937664 radius=0.5426888053709441
- added link 24, mass 0.3931597829033822; collision cylinder length=0.42493009252937664 radius=0.5426888053709441; visual cylinder length=0.42493009252937664 radius=0.5426888053709441
- link 0: mass 0.016562221436832083 -> 0.003919360339250734; geometry collision cylinder length=1.442823644237529 radius=0.02940532847591959; visual cylinder length=1.442823644237529 radius=0.02940532847591959
- link 11: mass 0.05843720197760504 -> 0.007085101111084106; geometry collision cylinder length=0.039176576910777916 radius=0.23993016166726788; visual cylinder length=0.039176576910777916 radius=0.23993016166726788
- link 22: mass 1.469920476335954 -> 0.3931597829033822; geometry collision cylinder length=0.42493009252937664 radius=0.5426888053709441; visual cylinder length=0.42493009252937664 radius=0.5426888053709441
Joints:
- removed joint 210_to_11
- removed joint 26_to_11
- removed joint 314_to_0
- removed joint 411_to_210
- removed joint 412_to_210
- removed joint 413_to_210
- removed joint 43_to_22
- removed joint 44_to_22
- removed joint 45_to_22
- removed joint 47_to_26
- removed joint 48_to_26
- removed joint 49_to_26
- added joint 23_to_11: type revolute, parent 11, child 23, origin xyz=0.18865344949164164 0.9109936564573404 0.3734537855485758 rpy=18.15343757858938 5.186843867187901 0.0, axis 0 0 1, limit lower=3.1415 upper=-3.1415 effort=1 velocity=1
- added joint 24_to_11: type revolute, parent 11, child 24, origin xyz=0.18865344949164164 0.9109936564573404 0.3734537855485758 rpy=24.204583438119172 5.186843867187901 0.0, axis 0 0 1, limit lower=3.1415 upper=-3.1415 effort=1 velocity=1
- joint 11_to_0: origin xyz=0.9739137415158122 0.9999 0.9753723564264214 rpy=6.623305055309696 2.0355958124422133 1.1957713899188829 -> xyz=0.8100042387937797 0.8497545831898448 0.8428329151479883 rpy=4.726851421616899 2.1332596079635504 5.241707572172651
- joint 22_to_11: axis 1 0 0 -> 0 0 1; origin xyz=0.9999 0.44850076168047337 0.26165231731438815 rpy=2.7437206674508094 2.2733772407708366 1.2236154125144392 -> xyz=0.18865344949164164 0.9109936564573404 0.3734537855485758 rpy=12.102291719059586 5.186843867187901 0.0
